File: sequencer-pcb/sequencer-pcb.sch (KiCad schematic (older format))
At the start: 59 parts, among them J1 Ribbon, J2 Conn_02x10_Counter_Clockwise, J3 Conn_01x02_Female, SW1 SW_Push, SW10 SW_Push, SW11 SW_Push, SW12 SW_Push, SW13 SW_Push, SW2 SW_Push, SW3 SW_Push, SW4 SW_Push, SW5 SW_Push, SW6 SW_Push, SW7 SW_Push, SW8 SW_Push, SW9 SW_Push

Commit message: kicad updates
Parts:
- RV1, RV10, RV11, RV2, RV3, RV4, RV5, RV6, RV7, RV8, RV9: footprint Potentiometer_THT:Potentiometer_Alps_RK09K_Single_Vertical -> Potentiometer_THT:Potentiometer_Bourns_PTV09A-1_Single_Vertical
- SW1, SW10, SW11, SW12, SW13, SW2, SW3, SW4, SW5, SW6, SW7, SW8, SW9: footprint Button_Switch_THT:SW_PUSH_6mm -> Button_Switch_THT:SW_PUSH_6mm_H5mm
Changed lines of the file:
@@
 F 0 "SW1" H 4250 3635 50  0000 C CNN
 F 1 "SW_Push" H 4250 3544 50  0000 C CNN
-F 2 "Button_Switch_THT:SW_PUSH_6mm" H 4250 3550 50  0001 C CNN
+F 2 "Button_Switch_THT:SW_PUSH_6mm_H5mm" H 4250 3550 50  0001 C CNN
 F 3 "~" H 4250 3550 50  0001 C CNN
 	1    4250 3350
@@
 F 0 "SW3" H 4850 3635 50  0000 C CNN
 F 1 "SW_Push" H 4850 3544 50  0000 C CNN
-F 2 "Button_Switch_THT:SW_PUSH_6mm" H 4850 3550 50  0001 C CNN
+F 2 "Button_Switch_THT:SW_PUSH_6mm_H5mm" H 4850 3550 50  0001 C CNN
 F 3 "~" H 4850 3550 50  0001 C CNN
 	1    4850 3350
@@
 F 0 "SW7" H 5850 3635 50  0000 C CNN
 F 1 "SW_Push" H 5850 3544 50  0000 C CNN
-F 2 "Button_Switch_THT:SW_PUSH_6mm" H 5850 3550 50  0001 C CNN
+F 2 "Button_Switch_THT:SW_PUSH_6mm_H5mm" H 5850 3550 50  0001 C CNN
 F 3 "~" H 5850 3550 50  0001 C CNN
 	1    5850 3350
@@
 F 0 "SW11" H 1450 5935 50  0000 C CNN
 F 1 "SW_Push" H 1450 5844 50  0000 C CNN
-F 2 "Button_Switch_THT:SW_PUSH_6mm" H 1450 5850 50  0001 C CNN
+F 2 "Button_Switch_THT:SW_PUSH_6mm_H5mm" H 1450 5850 50  0001 C CNN
 F 3 "~" H 1450 5850 50  0001 C CNN
 	1    1450 5650
@@
 F 0 "RV9" V 2093 4950 50  0000 C CNN
 F 1 "R_POT" V 2184 4950 50  0000 C CNN
-F 2 "Potentiometer_THT:Potentiometer_Alps_RK09K_Single_Vertical" H 2300 4950 50  0001 C CNN
+F 2 "Potentiometer_THT:Potentiometer_Bourns_PTV09A-1_Single_Vertical" H 2300 4950 50  0001 C CNN
 F 3 "~" H 2300 4950 50  0001 C CNN
 	1    2300 4950
@@
 F 0 "RV10" V 2743 4950 50  0000 C CNN
 F 1 "R_POT" V 2834 4950 50  0000 C CNN
-F 2 "Potentiometer_THT:Potentiometer_Alps_RK09K_Single_Vertical" H 2950 4950 50  0001 C CNN
+F 2 "Potentiometer_THT:Potentiometer_Bourns_PTV09A-1_Single_Vertical" H 2950 4950 50  0001 C CNN
 F 3 "~" H 2950 4950 50  0001 C CNN
 	1    2950 4950
@@
 F 0 "RV8" V 5885 1950 50  0000 C CNN
 F 1 "100k" V 5794 1950 50  0000 C CNN
-F 2 "Potentiometer_THT:Potentiometer_Alps_RK09K_Single_Vertical" H 6000 1950 50  0001 C CNN
+F 2 "Potentiometer_THT:Potentiometer_Bourns_PTV09A-1_Single_Vertical" H 6000 1950 50  0001 C CNN
 F 3 "~" H 6000 1950 50  0001 C CNN
 	1    6000 1950
@@
 F 0 "RV7" V 5135 1950 50  0000 C CNN
 F 1 "100k" V 5044 1950 50  0000 C CNN
-F 2 "Potentiometer_THT:Potentiometer_Alps_RK09K_Single_Vertical" H 5250 1950 50  0001 C CNN
+F 2 "Potentiometer_THT:Potentiometer_Bourns_PTV09A-1_Single_Vertical" H 5250 1950 50  0001 C CNN
 F 3 "~" H 5250 1950 50  0001 C CNN
 	1    5250 1950
@@
 F 0 "RV6" V 4335 1950 50  0000 C CNN
 F 1 "100k" V 4244 1950 50  0000 C CNN
-F 2 "Potentiometer_THT:Potentiometer_Alps_RK09K_Single_Vertical" H 4450 1950 50  0001 C CNN
+F 2 "Potentiometer_THT:Potentiometer_Bourns_PTV09A-1_Single_Vertical" H 4450 1950 50  0001 C CNN
 F 3 "~" H 4450 1950 50  0001 C CNN
 	1    4450 1950
@@
 F 0 "RV5" V 3535 1950 50  0000 C CNN
 F 1 "100k" V 3444 1950 50  0000 C CNN
-F 2 "Potentiometer_THT:Potentiometer_Alps_RK09K_Single_Vertical" H 3650 1950 50  0001 C CNN
+F 2 "Potentiometer_THT:Potentiometer_Bourns_PTV09A-1_Single_Vertical" H 3650 1950 50  0001 C CNN
 F 3 "~" H 3650 1950 50  0001 C CNN
 	1    3650 1950
@@
 F 0 "RV4" V 5793 1300 50  0000 C CNN
 F 1 "100k" V 5884 1300 50  0000 C CNN
-F 2 "Potentiometer_THT:Potentiometer_Alps_RK09K_Single_Vertical" H 6000 1300 50  0001 C CNN
+F 2 "Potentiometer_THT:Potentiometer_Bourns_PTV09A-1_Single_Vertical" H 6000 1300 50  0001 C CNN
 F 3 "~" H 6000 1300 50  0001 C CNN
 	1    6000 1300
@@
 F 0 "RV3" V 5043 1300 50  0000 C CNN
 F 1 "100k" V 5134 1300 50  0000 C CNN
-F 2 "Potentiometer_THT:Potentiometer_Alps_RK09K_Single_Vertical" H 5250 1300 50  0001 C CNN
+F 2 "Potentiometer_THT:Potentiometer_Bourns_PTV09A-1_Single_Vertical" H 5250 1300 50  0001 C CNN
 F 3 "~" H 5250 1300 50  0001 C CNN
 	1    5250 1300
@@
 F 0 "RV2" V 4193 1300 50  0000 C CNN
 F 1 "100k" V 4284 1300 50  0000 C CNN
-F 2 "Potentiometer_THT:Potentiometer_Alps_RK09K_Single_Vertical" H 4400 1300 50  0001 C CNN
+F 2 "Potentiometer_THT:Potentiometer_Bourns_PTV09A-1_Single_Vertical" H 4400 1300 50  0001 C CNN
 F 3 "~" H 4400 1300 50  0001 C CNN
 	1    4400 1300
@@
 F 0 "RV1" V 3443 1300 50  0000 C CNN
 F 1 "100k" V 3534 1300 50  0000 C CNN
-F 2 "Potentiometer_THT:Potentiometer_Alps_RK09K_Single_Vertical" H 3650 1300 50  0001 C CNN
+F 2 "Potentiometer_THT:Potentiometer_Bourns_PTV09A-1_Single_Vertical" H 3650 1300 50  0001 C CNN
 F 3 "~" H 3650 1300 50  0001 C CNN
 	1    3650 1300
@@
 F 0 "SW8" H 5850 4335 50  0000 C CNN
 F 1 "SW_Push" H 5850 4244 50  0000 C CNN
-F 2 "Button_Switch_THT:SW_PUSH_6mm" H 5850 4250 50  0001 C CNN
+F 2 "Button_Switch_THT:SW_PUSH_6mm_H5mm" H 5850 4250 50  0001 C CNN
 F 3 "~" H 5850 4250 50  0001 C CNN
 	1    5850 4050
@@
 F 0 "SW6" H 5350 4335 50  0000 C CNN
 F 1 "SW_Push" H 5350 4244 50  0000 C CNN
-F 2 "Button_Switch_THT:SW_PUSH_6mm" H 5350 4250 50  0001 C CNN
+F 2 "Button_Switch_THT:SW_PUSH_6mm_H5mm" H 5350 4250 50  0001 C CNN
 F 3 "~" H 5350 4250 50  0001 C CNN
 	1    5350 4050
@@
 F 0 "SW4" H 4850 4335 50  0000 C CNN
 F 1 "SW_Push" H 4850 4244 50  0000 C CNN
-F 2 "Button_Switch_THT:SW_PUSH_6mm" H 4850 4250 50  0001 C CNN
+F 2 "Button_Switch_THT:SW_PUSH_6mm_H5mm" H 4850 4250 50  0001 C CNN
 F 3 "~" H 4850 4250 50  0001 C CNN
 	1    4850 4050
@@
 F 0 "SW2" H 4250 4335 50  0000 C CNN
 F 1 "SW_Push" H 4250 4244 50  0000 C CNN
-F 2 "Button_Switch_THT:SW_PUSH_6mm" H 4250 4250 50  0001 C CNN
+F 2 "Button_Switch_THT:SW_PUSH_6mm_H5mm" H 4250 4250 50  0001 C CNN
 F 3 "~" H 4250 4250 50  0001 C CNN
 	1    4250 4050
@@
 F 0 "SW10" H 1450 6335 50  0000 C CNN
 F 1 "SW_Push" H 1450 6244 50  0000 C CNN
-F 2 "Button_Switch_THT:SW_PUSH_6mm" H 1450 6250 50  0001 C CNN
+F 2 "Button_Switch_THT:SW_PUSH_6mm_H5mm" H 1450 6250 50  0001 C CNN
 F 3 "~" H 1450 6250 50  0001 C CNN
 	1    1450 6050
@@
 F 0 "SW9" H 1450 6685 50  0000 C CNN
 F 1 "SW_Push" H 1450 6594 50  0000 C CNN
-F 2 "Button_Switch_THT:SW_PUSH_6mm" H 1450 6600 50  0001 C CNN
+F 2 "Button_Switch_THT:SW_PUSH_6mm_H5mm" H 1450 6600 50  0001 C CNN
 F 3 "~" H 1450 6600 50  0001 C CNN
 	1    1450 6400
@@
 F 0 "SW5" H 5350 3635 50  0000 C CNN
 F 1 "SW_Push" H 5350 3544 50  0000 C CNN
-F 2 "Button_Switch_THT:SW_PUSH_6mm" H 5350 3550 50  0001 C CNN
+F 2 "Button_Switch_THT:SW_PUSH_6mm_H5mm" H 5350 3550 50  0001 C CNN
 F 3 "~" H 5350 3550 50  0001 C CNN
 	1    5350 3350
@@
 F 0 "SW13" H 1450 5585 50  0000 C CNN
 F 1 "SW_Push" H 1450 5494 50  0000 C CNN
-F 2 "Button_Switch_THT:SW_PUSH_6mm" H 1450 5500 50  0001 C CNN
+F 2 "Button_Switch_THT:SW_PUSH_6mm_H5mm" H 1450 5500 50  0001 C CNN
 F 3 "~" H 1450 5500 50  0001 C CNN
 	1    1450 5300
@@
 F 0 "SW12" H 1450 5185 50  0000 C CNN
 F 1 "SW_Push" H 1450 5094 50  0000 C CNN
-F 2 "Button_Switch_THT:SW_PUSH_6mm" H 1450 5100 50  0001 C CNN
+F 2 "Button_Switch_THT:SW_PUSH_6mm_H5mm" H 1450 5100 50  0001 C CNN
 F 3 "~" H 1450 5100 50  0001 C CNN
 	1    1450 4900
@@
 F 0 "RV11" V 2443 5450 50  0000 C CNN
 F 1 "R_POT" V 2534 5450 50  0000 C CNN
-F 2 "Potentiometer_THT:Potentiometer_Alps_RK09K_Single_Vertical" H 2650 5450 50  0001 C CNN
+F 2 "Potentiometer_THT:Potentiometer_Bourns_PTV09A-1_Single_Vertical" H 2650 5450 50  0001 C CNN
 F 3 "~" H 2650 5450 50  0001 C CNN
 	1    2650 5450
