File: sequencer-pcb/sequencer-pcb.sch (KiCad schematic (older format))
At the start: 59 parts, among them J1 Ribbon, J2 Conn_02x10_Counter_Clockwise, J3 Conn_01x02_Female, SW1 SW_Push, SW10 SW_Push, SW11 SW_Push, SW12 SW_Push, SW13 SW_Push, SW2 SW_Push, SW3 SW_Push, SW4 SW_Push, SW5 SW_Push, SW6 SW_Push, SW7 SW_Push, SW8 SW_Push, SW9 SW_Push

Commit message: new pcb
Parts:
- added OLED_Display1: OLED, Display:OLED_SPI_128x32, symbol Display_Character:OLED
- added R18, R19, R20, R21, R22: R, Resistor_SMD:R_1806_4516Metric_Pad1.57x1.80mm_HandSolder, symbol Device:R
- added TP1: TestPoint, TestPoint:TestPoint_THTPad_2.5x2.5mm_Drill1.2mm, symbol Connector:TestPoint
- J3: value Conn_01x02_Female -> Conn_01x03_Female; footprint Connector_PinHeader_2.54mm:PinHeader_1x02_P2.54mm_Vertical -> Connector_PinHeader_2.54mm:PinHeader_1x03_P2.54mm_Vertical; symbol Connector:Conn_01x02_Female -> Connector:Conn_01x03_Female
- renumbered RV9 to SP1, RV10 to SP2, RV11 to SP3, SW12 to SSW1, SW10 to SSW2, SW11 to SSW3, SW9 to SSW4, SW13 to SSW5, TP6 to TP2, TP5 to TP3
Connections:
- net labels added: +3.3V, CLK, CS, DC, MOSI, RES, SP1, SP2, SP3, SSW1, SSW2, SSW3, SSW4, SSW5
- net labels removed: NC
- wire segments 90 -> 121
Other:
- note added: "Setting \npotentiometers"
- note added: "Setting switches\n"
- moved on the sheet: SP1, SP2, SP3, SSW1, SSW2, SSW3, SSW4, SSW5

Commit message: new led
Parts:
- D9: footprint LED_THT:LED_D5.0mm -> LED_SMD:LED_1206_3216Metric_Pad1.42x1.75mm_HandSolder
- OLED_Display1: symbol Display_Character:OLED -> sequencer-pcb-rescue:OLED-Display_Character
Changed lines of the file:
@@
 F 0 "D9" H 2243 1366 50  0000 C CNN
 F 1 "LED" H 2243 1275 50  0000 C CNN
-F 2 "LED_THT:LED_D5.0mm" H 2250 1150 50  0001 C CNN
+F 2 "LED_SMD:LED_1206_3216Metric_Pad1.42x1.75mm_HandSolder" H 2250 1150 50  0001 C CNN
 F 3 "~" H 2250 1150 50  0001 C CNN
 	1    2250 1150
@@
 R1
 $Comp
-L Display_Character:OLED OLED_Display1
+L sequencer-pcb-rescue:OLED-Display_Character OLED_Display1
 U 1 1 5F4AFC7D
 P 5250 6250

Commit message: new led
Parts:
- R1, R10, R11, R12, R13, R14, R15, R16, R17, R18, R19, R2, R20, R21, R22, R3, R4, R5, R6, R7, R8, R9: footprint Resistor_SMD:R_1806_4516Metric_Pad1.57x1.80mm_HandSolder -> Resistor_SMD:R_1206_3216Metric_Pad1.42x1.75mm_HandSolder
- RV1, RV2, RV3, RV4, RV5, RV6, RV7, RV8, SP1, SP2, SP3: footprint Potentiometer_THT:Potentiometer_Bourns_PTV09A-1_Single_Vertical -> Potentiometer_THT:Potentiometer_Alps_RK09K_Single_Vertical

Commit message: boms
Parts:
- R1, R10, R11, R14, R15, R2, R5, R6, R9: value R -> 220
- R12, R13, R16, R17, R18, R19, R20, R21, R22, R3, R4, R7, R8: value R -> 10k
- SP1, SP2, SP3: value R_POT -> R_POT_SETTING
Changed lines of the file:
@@
 P 1750 1150
 F 0 "R9" V 1543 1150 50  0000 C CNN
-F 1 "R" V 1634 1150 50  0000 C CNN
+F 1 "220" V 1634 1150 50  0000 C CNN
 F 2 "Resistor_SMD:R_1206_3216Metric_Pad1.42x1.75mm_HandSolder" V 1680 1150 50  0001 C CNN
 F 3 "~" H 1750 1150 50  0001 C CNN
@@
 P 1150 2250
 F 0 "R1" H 1220 2296 50  0000 L CNN
-F 1 "R" H 1220 2205 50  0000 L CNN
+F 1 "220" H 1220 2205 50  0000 L CNN
 F 2 "Resistor_SMD:R_1206_3216Metric_Pad1.42x1.75mm_HandSolder" V 1080 2250 50  0001 C CNN
 F 3 "~" H 1150 2250 50  0001 C CNN
@@
 P 1700 2250
 F 0 "R5" H 1770 2296 50  0000 L CNN
-F 1 "R" H 1770 2205 50  0000 L CNN
+F 1 "220" H 1770 2205 50  0000 L CNN
 F 2 "Resistor_SMD:R_1206_3216Metric_Pad1.42x1.75mm_HandSolder" V 1630 2250 50  0001 C CNN
 F 3 "~" H 1700 2250 50  0001 C CNN
@@
 P 2200 2250
 F 0 "R10" H 2270 2296 50  0000 L CNN
-F 1 "R" H 2270 2205 50  0000 L CNN
+F 1 "220" H 2270 2205 50  0000 L CNN
 F 2 "Resistor_SMD:R_1206_3216Metric_Pad1.42x1.75mm_HandSolder" V 2130 2250 50  0001 C CNN
 F 3 "~" H 2200 2250 50  0001 C CNN
@@
 P 2750 2250
 F 0 "R14" H 2820 2296 50  0000 L CNN
-F 1 "R" H 2820 2205 50  0000 L CNN
+F 1 "220" H 2820 2205 50  0000 L CNN
 F 2 "Resistor_SMD:R_1206_3216Metric_Pad1.42x1.75mm_HandSolder" V 2680 2250 50  0001 C CNN
 F 3 "~" H 2750 2250 50  0001 C CNN
@@
 P 1150 3550
 F 0 "R2" H 1220 3596 50  0000 L CNN
-F 1 "R" H 1220 3505 50  0000 L CNN
+F 1 "220" H 1220 3505 50  0000 L CNN
 F 2 "Resistor_SMD:R_1206_3216Metric_Pad1.42x1.75mm_HandSolder" V 1080 3550 50  0001 C CNN
 F 3 "~" H 1150 3550 50  0001 C CNN
@@
 P 1700 3550
 F 0 "R6" H 1770 3596 50  0000 L CNN
-F 1 "R" H 1770 3505 50  0000 L CNN
+F 1 "220" H 1770 3505 50  0000 L CNN
 F 2 "Resistor_SMD:R_1206_3216Metric_Pad1.42x1.75mm_HandSolder" V 1630 3550 50  0001 C CNN
 F 3 "~" H 1700 3550 50  0001 C CNN
@@
 P 2200 3550
 F 0 "R11" H 2270 3596 50  0000 L CNN
-F 1 "R" H 2270 3505 50  0000 L CNN
+F 1 "220" H 2270 3505 50  0000 L CNN
 F 2 "Resistor_SMD:R_1206_3216Metric_Pad1.42x1.75mm_HandSolder" V 2130 3550 50  0001 C CNN
 F 3 "~" H 2200 3550 50  0001 C CNN
@@
 P 2750 3550
 F 0 "R15" H 2820 3596 50  0000 L CNN
-F 1 "R" H 2820 3505 50  0000 L CNN
+F 1 "220" H 2820 3505 50  0000 L CNN
 F 2 "Resistor_SMD:R_1206_3216Metric_Pad1.42x1.75mm_HandSolder" V 2680 3550 50  0001 C CNN
 F 3 "~" H 2750 3550 50  0001 C CNN
@@
 P 4250 2950
 F 0 "R3" H 4320 2996 50  0000 L CNN
-F 1 "R" H 4320 2905 50  0000 L CNN
+F 1 "10k" H 4320 2905 50  0000 L CNN
 F 2 "Resistor_SMD:R_1206_3216Metric_Pad1.42x1.75mm_HandSolder" V 4180 2950 50  0001 C CNN
 F 3 "~" H 4250 2950 50  0001 C CNN
@@
 P 4850 2950
 F 0 "R7" H 4920 2996 50  0000 L CNN
-F 1 "R" H 4920 2905 50  0000 L CNN
+F 1 "10k" H 4920 2905 50  0000 L CNN
 F 2 "Resistor_SMD:R_1206_3216Metric_Pad1.42x1.75mm_HandSolder" V 4780 2950 50  0001 C CNN
 F 3 "~" H 4850 2950 50  0001 C CNN
@@
 P 5850 2950
 F 0 "R16" H 5920 2996 50  0000 L CNN
-F 1 "R" H 5920 2905 50  0000 L CNN
+F 1 "10k" H 5920 2905 50  0000 L CNN
 F 2 "Resistor_SMD:R_1206_3216Metric_Pad1.42x1.75mm_HandSolder" V 5780 2950 50  0001 C CNN
 F 3 "~" H 5850 2950 50  0001 C CNN
@@
 P 4250 4450
 F 0 "R4" H 4320 4496 50  0000 L CNN
-F 1 "R" H 4320 4405 50  0000 L CNN
+F 1 "10k" H 4320 4405 50  0000 L CNN
 F 2 "Resistor_SMD:R_1206_3216Metric_Pad1.42x1.75mm_HandSolder" V 4180 4450 50  0001 C CNN
 F 3 "~" H 4250 4450 50  0001 C CNN
@@
 P 4850 4450
 F 0 "R8" H 4920 4496 50  0000 L CNN
-F 1 "R" H 4920 4405 50  0000 L CNN
+F 1 "10k" H 4920 4405 50  0000 L CNN
 F 2 "Resistor_SMD:R_1206_3216Metric_Pad1.42x1.75mm_HandSolder" V 4780 4450 50  0001 C CNN
 F 3 "~" H 4850 4450 50  0001 C CNN
@@
 P 5350 4450
 F 0 "R13" H 5420 4496 50  0000 L CNN
-F 1 "R" H 5420 4405 50  0000 L CNN
+F 1 "10k" H 5420 4405 50  0000 L CNN
 F 2 "Resistor_SMD:R_1206_3216Metric_Pad1.42x1.75mm_HandSolder" V 5280 4450 50  0001 C CNN
 F 3 "~" H 5350 4450 50  0001 C CNN
@@
 P 5850 4450
 F 0 "R17" H 5920 4496 50  0000 L CNN
-F 1 "R" H 5920 4405 50  0000 L CNN
+F 1 "10k" H 5920 4405 50  0000 L CNN
 F 2 "Resistor_SMD:R_1206_3216Metric_Pad1.42x1.75mm_HandSolder" V 5780 4450 50  0001 C CNN
 F 3 "~" H 5850 4450 50  0001 C CNN
@@
 P 5350 2950
 F 0 "R12" H 5420 2996 50  0000 L CNN
-F 1 "R" H 5420 2905 50  0000 L CNN
+F 1 "10k" H 5420 2905 50  0000 L CNN
 F 2 "Resistor_SMD:R_1206_3216Metric_Pad1.42x1.75mm_HandSolder" V 5280 2950 50  0001 C CNN
 F 3 "~" H 5350 2950 50  0001 C CNN
@@
 P 2350 4900
 F 0 "SP3" H 2350 4650 50  0000 C CNN
-F 1 "R_POT" H 2350 4550 50  0000 C CNN
+F 1 "R_POT_SETTING" H 2350 4550 50  0000 C CNN
 F 2 "Potentiometer_THT:Potentiometer_Alps_RK09K_Single_Vertical" H 2350 4900 50  0001 C CNN
 F 3 "~" H 2350 4900 50  0001 C CNN
@@
 P 1950 4900
 F 0 "SP2" H 1900 4650 50  0000 C CNN
-F 1 "R_POT" H 1900 4550 50  0000 C CNN
+F 1 "R_POT_SETTING" H 1900 4550 50  0000 C CNN
 F 2 "Potentiometer_THT:Potentiometer_Alps_RK09K_Single_Vertical" H 1950 4900 50  0001 C CNN
 F 3 "~" H 1950 4900 50  0001 C CNN
@@
 P 1550 4900
 F 0 "SP1" H 1500 4650 50  0000 C CNN
-F 1 "R_POT" H 1500 4550 50  0000 C CNN
+F 1 "R_POT_SETTING" H 1500 4550 50  0000 C CNN
 F 2 "Potentiometer_THT:Potentiometer_Alps_RK09K_Single_Vertical" H 1550 4900 50  0001 C CNN
 F 3 "~" H 1550 4900 50  0001 C CNN
@@
 P 1300 6100
 F 0 "R18" H 1370 6146 50  0000 L CNN
-F 1 "R" H 1370 6055 50  0000 L CNN
+F 1 "10k" H 1370 6055 50  0000 L CNN
 F 2 "Resistor_SMD:R_1206_3216Metric_Pad1.42x1.75mm_HandSolder" V 1230 6100 50  0001 C CNN
 F 3 "~" H 1300 6100 50  0001 C CNN
@@
 P 1800 6100
 F 0 "R20" H 1870 6146 50  0000 L CNN
-F 1 "R" H 1870 6055 50  0000 L CNN
+F 1 "10k" H 1870 6055 50  0000 L CNN
 F 2 "Resistor_SMD:R_1206_3216Metric_Pad1.42x1.75mm_HandSolder" V 1730 6100 50  0001 C CNN
 F 3 "~" H 1800 6100 50  0001 C CNN
@@
 P 2300 6100
 F 0 "R21" H 2370 6146 50  0000 L CNN
-F 1 "R" H 2370 6055 50  0000 L CNN
+F 1 "10k" H 2370 6055 50  0000 L CNN
 F 2 "Resistor_SMD:R_1206_3216Metric_Pad1.42x1.75mm_HandSolder" V 2230 6100 50  0001 C CNN
 F 3 "~" H 2300 6100 50  0001 C CNN
@@
 P 2750 6100
 F 0 "R22" H 2820 6146 50  0000 L CNN
-F 1 "R" H 2820 6055 50  0000 L CNN
+F 1 "10k" H 2820 6055 50  0000 L CNN
 F 2 "Resistor_SMD:R_1206_3216Metric_Pad1.42x1.75mm_HandSolder" V 2680 6100 50  0001 C CNN
 F 3 "~" H 2750 6100 50  0001 C CNN
@@
 P 1300 7550
 F 0 "R19" H 1370 7596 50  0000 L CNN
-F 1 "R" H 1370 7505 50  0000 L CNN
+F 1 "10k" H 1370 7505 50  0000 L CNN
 F 2 "Resistor_SMD:R_1206_3216Metric_Pad1.42x1.75mm_HandSolder" V 1230 7550 50  0001 C CNN
 F 3 "~" H 1300 7550 50  0001 C CNN

Commit message: new pcb
Parts:
- removed R22: 10k, Resistor_SMD:R_1206_3216Metric_Pad1.42x1.75mm_HandSolder, symbol Device:R
- removed SP2: R_POT_SETTING, Potentiometer_THT:Potentiometer_Alps_RK09K_Single_Vertical, symbol Device:R_POT
- removed SSW2, SSW4: SW_Push, Button_Switch_THT:SW_PUSH_6mm_H5mm, symbol Switch:SW_Push
- added SW9: Rotary_Encoder_Switch, Rotary_Encoder:RotaryEncoder_Alps_EC12E-Switch_Vertical_H20mm, symbol Device:Rotary_Encoder_Switch
- R12, R13, R16, R17, R18, R19, R20, R21, R3, R4, R7, R8: value 10k -> 2k2
- renumbered SSW5 to SSW2
Connections:
- net +3V3: now also SW9.S2
- net GND: now also R19.1, SW9.C; no longer R19.2
- net SSW1: now also J1.9 (Pin_9); no longer J1.10 (Pin_10)
- net SSW2: now also J1.11 (Pin_11); no longer J1.14 (Pin_14)
- net SSW4: now also J1.14 (Pin_14), R19.2, SW9.S1; no longer J1.9 (Pin_9)
- net SP2 renamed RE2
- net RE2: now also SW9.A
- removed net SSW5: J1.11 (Pin_11), R19.1
- new net RE1: J1.10 (Pin_10), SW9.B
Other:
- moved on the sheet: OLED_Display1

Commit message: cv expander
Parts:
- R9: value 220 -> 1k
Changed lines of the file:
@@
 P 1750 1150
 F 0 "R9" V 1543 1150 50  0000 C CNN
-F 1 "220" V 1634 1150 50  0000 C CNN
+F 1 "1k" V 1634 1150 50  0000 C CNN
 F 2 "Resistor_SMD:R_1206_3216Metric_Pad1.42x1.75mm_HandSolder" V 1680 1150 50  0001 C CNN
 F 3 "~" H 1750 1150 50  0001 C CNN
