File: sequencer-pcb/controller.sch (KiCad schematic (older format))
At the start: 21 parts

Commit message: boms
Parts:
- removed J?: Conn_02x08_Counter_Clockwise, symbol Connector_Generic:Conn_02x08_Counter_Clockwise
- removed J?: Conn_02x10_Counter_Clockwise, symbol Connector_Generic:Conn_02x10_Counter_Clockwise
- added J?: Ribbon, Connector_IDC:IDC-Header_2x10_P2.54mm_Vertical, symbol Connector_Generic:Conn_02x10_Counter_Clockwise
- added J?: Conn_02x10_Counter_Clockwise, Connector_IDC:IDC-Header_2x10_P2.54mm_Vertical, symbol Connector_Generic:Conn_02x10_Counter_Clockwise
- J? (x2): value Conn_01x17_Male -> Conn_01x20_Male
Connections:
- net +5V: now also J?.4 (Pin_4)
- net B1: now also J?.14 (Pin_14)
- net B2: now also J?.13 (Pin_13)
- net B3: now also J?.8 (Pin_8)
- net B4: now also J?.7 (Pin_7)
- net B5: now also J?.20 (Pin_20)
- net B6: now also J?.19 (Pin_19)
- net B7: now also J?.20 (Pin_20)
- net B8: now also J?.19 (Pin_19)
- net GND: now also J?.2 (Pin_2)
- net L1: now also J?.10 (Pin_10)
- net L2: now also J?.9 (Pin_9)
- net L3: now also J?.4 (Pin_4)
- net L4: now also J?.3 (Pin_3)
- net L5: now also J?.16 (Pin_16)
- net L6: now also J?.15 (Pin_15)
- net L7: now also J?.16 (Pin_16)
- net L8: now also J?.15 (Pin_15)
- net R1: now also J?.12 (Pin_12)
- net R2: now also J?.11 (Pin_11)
- net R3: now also J?.6 (Pin_6)
- net R4: now also J?.5 (Pin_5)
- net R5: now also J?.18 (Pin_18)
- net R6: now also J?.17 (Pin_17)
- net R7: now also J?.18 (Pin_18)
- net R8: now also J?.17 (Pin_17)
- new net +3V3: J?.13 (Pin_13)
- new net CLK: J?.3 (Pin_3)
- new net CS: J?.8 (Pin_8)
- new net DC: J?.7 (Pin_7)
- new net MOSI: J?.5 (Pin_5)
- new net RES: J?.6 (Pin_6)
- new net SP1: J?.2 (Pin_2)
- new net SP2: J?.1 (Pin_1)
- new net SP3: J?.1 (Pin_1)
- new net SSW1: J?.10 (Pin_10)
- new net SSW2: J?.14 (Pin_14)
- new net SSW3: J?.12 (Pin_12)
- new net SSW4: J?.9 (Pin_9)
- new net SSW5: J?.11 (Pin_11)
Other:
- note added: "Ribbon (IDC) connections"
- moved on the sheet: J?, TP?
