File: sequencer-pcb/cv_expander.sch (KiCad schematic (older format))
At the start: 16 parts, among them J1 Conn_01x20_Male, J10 VCO Exp in, J11 VCF Aud in, J12 Trig Out, J13 EG out, J14 VCF Out, J2 VCA In, J3 VCO Lin In, J4 LFO In, J5 KB CV out, J6 Gate out, J7 LFO Out, J8 VCO out, J9 VCF In

Commit message: sequencer
Parts:
- removed H2: MountingHole_GND, MountingHole:MountingHole_2.7mm_M2.5_Pad, symbol Mechanical:MountingHole_Pad
- removed J4: LFO In, symbol Connector:AudioJack2
- added J6: LFO in, Connector_Audio:3.5mm_Electrokit, symbol Connector:AudioJack3-mono
- added TP1: TestPoint, TestPoint:TestPoint_Plated_Hole_D2.0mm, symbol Connector:TestPoint
- added TP2: TestPoint, TestPoint:TestPoint_Pad_2.0x2.0mm, symbol Connector:TestPoint
- J10: renamed from J6; footprint (none) -> Connector_Audio:3.5mm_Electrokit; symbol Connector:AudioJack3 -> Connector:AudioJack3-mono
- J11: renamed from J13; footprint (none) -> Connector_Audio:3.5mm_Electrokit; symbol Connector:AudioJack3 -> Connector:AudioJack3-mono
- J12: renamed from J7; footprint (none) -> Connector_Audio:3.5mm_Electrokit; symbol Connector:AudioJack3 -> Connector:AudioJack3-mono
- J13: renamed from J14; footprint (none) -> Connector_Audio:3.5mm_Electrokit; symbol Connector:AudioJack3 -> Connector:AudioJack3-mono
- J14: renamed from J8; footprint (none) -> Connector_Audio:3.5mm_Electrokit; symbol Connector:AudioJack3 -> Connector:AudioJack3-mono
- J2: footprint (none) -> Connector_Audio:3.5mm_Electrokit; symbol Connector:AudioJack3 -> Connector:AudioJack3-mono
- J3: renamed from J9; footprint (none) -> Connector_Audio:3.5mm_Electrokit; symbol Connector:AudioJack3 -> Connector:AudioJack3-mono
- J4: renamed from J3; footprint (none) -> Connector_Audio:3.5mm_Electrokit; symbol Connector:AudioJack3 -> Connector:AudioJack3-mono
- J5: renamed from J10; footprint (none) -> Connector_Audio:3.5mm_Electrokit; symbol Connector:AudioJack3 -> Connector:AudioJack3-mono
- J7: renamed from J11; footprint (none) -> Connector_Audio:3.5mm_Electrokit; symbol Connector:AudioJack3 -> Connector:AudioJack3-mono
- J8: renamed from J5; footprint (none) -> Connector_Audio:3.5mm_Electrokit; symbol Connector:AudioJack3 -> Connector:AudioJack3-mono
- J9: renamed from J12; footprint (none) -> Connector_Audio:3.5mm_Electrokit; symbol Connector:AudioJack3 -> Connector:AudioJack3-mono

Commit message: new pcb
Parts:
- J10, J11, J12, J13, J14, J2, J3, J4, J5, J6, J7, J8, J9: symbol Connector:AudioJack3-mono -> cv_expander-rescue:AudioJack3-mono-Connector
Changed lines of the file:
@@
 $EndComp
 $Comp
-L Connector:AudioJack3-mono J2
+L cv_expander-rescue:AudioJack3-mono-Connector J2
 U 1 1 5F45E3E2
 P 7250 2050
@@
 $EndComp
 $Comp
-L Connector:AudioJack3-mono J3
+L cv_expander-rescue:AudioJack3-mono-Connector J3
 U 1 1 5F45E3E8
 P 8100 2300
@@
 	6700 2800 6700 2850
 $Comp
-L Connector:AudioJack3-mono J5
+L cv_expander-rescue:AudioJack3-mono-Connector J5
 U 1 1 5F45E3F4
 P 8300 2750
@@
 $EndComp
 $Comp
-L Connector:AudioJack3-mono J8
+L cv_expander-rescue:AudioJack3-mono-Connector J8
 U 1 1 5F45E406
 P 7250 3550
@@
 $EndComp
 $Comp
-L Connector:AudioJack3-mono J9
+L cv_expander-rescue:AudioJack3-mono-Connector J9
 U 1 1 5F45E40C
 P 8350 3650
@@
 $EndComp
 $Comp
-L Connector:AudioJack3-mono J11
+L cv_expander-rescue:AudioJack3-mono-Connector J11
 U 1 1 5F45E418
 P 8350 4150
@@
 $EndComp
 $Comp
-L Connector:AudioJack3-mono J12
+L cv_expander-rescue:AudioJack3-mono-Connector J12
 U 1 1 5F45E41E
 P 7250 4500
@@
 $EndComp
 $Comp
-L Connector:AudioJack3-mono J13
+L cv_expander-rescue:AudioJack3-mono-Connector J13
 U 1 1 5F45E424
 P 8350 4650
@@
 GND_D
 $Comp
-L Connector:AudioJack3-mono J14
+L cv_expander-rescue:AudioJack3-mono-Connector J14
 U 1 1 5F48864B
 P 7250 5000
@@
 GND_D
 $Comp
-L Connector:AudioJack3-mono J10
+L cv_expander-rescue:AudioJack3-mono-Connector J10
 U 1 1 5F45E412
 P 7250 4000
@@
 $EndComp
 $Comp
-L Connector:AudioJack3-mono J6
+L cv_expander-rescue:AudioJack3-mono-Connector J6
 U 1 1 5F449E33
 P 7250 3100
@@
 GND_D
 $Comp
-L Connector:AudioJack3-mono J7
+L cv_expander-rescue:AudioJack3-mono-Connector J7
 U 1 1 5F45E400
 P 8350 3200
@@
 	6250 4900 6250 4350
 $Comp
-L Connector:AudioJack3-mono J4
+L cv_expander-rescue:AudioJack3-mono-Connector J4
 U 1 1 5F45E3EE
 P 7250 2650

Commit message: cv expander
Parts:
- added H2: MountingHole_GND, MountingHole:MountingHole_2.7mm_M2.5_Pad, symbol Mechanical:MountingHole_Pad
Connections:
- net GND_D: now also H2.1
Changed lines of the file:
@@
 	-1   0    0    1
 $EndComp
+$Comp
+L Mechanical:MountingHole_Pad H2
+U 1 1 5F61DC1E
+P 4900 2600
+AR Path="/5F61DC1E" Ref="H2"  Part="1"
+AR Path="/5F450078/5F61DC1E" Ref="H?"  Part="1"
+F 0 "H2" V 4900 2750 50  0000 L CNN
+F 1 "MountingHole_GND" V 4800 2550 50  0000 L CNN
+F 2 "MountingHole:MountingHole_2.7mm_M2.5_Pad" H 4900 2600 50  0001 C CNN
+F 3 "~" H 4900 2600 50  0001 C CNN
+	1    4900 2600
+	0    -1   -1   0
+$EndComp
+Text GLabel 5000 2600 2    50   Input ~ 0
+GND_D
 $EndSCHEMATC
