File: sequencer-pcb/sequencer-pcb.kicad_pcb (KiCad board)
At the start: 2 copper layers, 56 parts, among them J1 Conn_02x08_Counter_Clockwise, J2 Conn_02x10_Counter_Clockwise, J3 Conn_01x02_Female, SW1 SW_Push, SW10 SW_Push, SW11 SW_Push, SW2 SW_Push, SW3 SW_Push, SW4 SW_Push, SW5 SW_Push, SW6 SW_Push, SW7 SW_Push, SW8 SW_Push, SW9 SW_Push

Commit message: updates
Parts:
- added RV11: R_POT, Potentiometer_THT:Potentiometer_Alps_RK09K_Single_Vertical, F.Cu at (189.2, 27.4)
- added SW12: SW_Push, Button_Switch_THT:SW_PUSH_6mm, F.Cu at (176.4, 31.2)
- added SW13: SW_Push, Button_Switch_THT:SW_PUSH_6mm, F.Cu at (88.1, 10.4)
- J1: value Conn_02x08_Counter_Clockwise -> Ribbon; footprint Connector_IDC:IDC-Header_2x08_P2.54mm_Vertical -> Connector_IDC:IDC-Header_2x10_P2.54mm_Vertical
- RV1, RV2, RV3, RV4, RV5, RV6, RV7, RV8: value R_POT -> 100k
- moved R7 50.2 mm to (140.2, 51.6), turned to 270 degrees
- moved SW9 28.0 mm to (176.3, 3.56), turned to 0 degrees
- moved R13 26.4 mm to (115.8, 0.76)
- moved R1 26.4 mm to (116.1, 9.75)
- moved R10 26.4 mm to (116.1, 14.5)
- moved R12 26.4 mm to (107.9, 10.1)
- moved R15 26.4 mm to (107.9, 14.9)
- moved R16 26.4 mm to (116.1, 19.2)
- moved R3 26.4 mm to (116.1, 5.00)
- moved R9 26.4 mm to (107.9, 5.39)
- moved R17 24.9 mm to (105.4, 26.9)
- moved D9 17.9 mm to (101.6, 10.7)
- moved SW10 17.8 mm to (176.3, 22.0), turned to 0 degrees
- moved J1 13.7 mm to (180.8, 45.5), turned to 180 degrees
- moved SW11 11.7 mm to (176.3, 12.8), turned to 0 degrees
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Connections:
- J1 pad 10: L7 -> L2
- J1 pad 11: L6 -> L3
- J1 pad 12: L5 -> L4
- J1 pad 13: L4 -> L5
- J1 pad 14: L3 -> L6
- J1 pad 15: L2 -> L7
- J1 pad 16: L1 -> L8
- J1 pad 9: L8 -> L1
- J2 pad 1: +5V -> B1
- J2 pad 10: B8 -> NC
- J2 pad 2: GND -> B2
- J2 pad 3: B1 -> B3
- J2 pad 4: B2 -> B4
- J2 pad 5: B3 -> B5
- J2 pad 6: B4 -> B6
- J2 pad 7: B5 -> B7
- J2 pad 8: B6 -> B8
- J2 pad 9: B7 -> NC

Commit message: kicad updates
Parts:
- RV1, RV10, RV11, RV2, RV3, RV4, RV5, RV6, RV7, RV8, RV9: footprint Potentiometer_THT:Potentiometer_Alps_RK09K_Single_Vertical -> Potentiometer_THT:Potentiometer_Bourns_PTV09A-1_Single_Vertical
- SW1, SW10, SW11, SW12, SW13, SW2, SW3, SW4, SW5, SW6, SW7, SW8, SW9: footprint Button_Switch_THT:SW_PUSH_6mm -> Button_Switch_THT:SW_PUSH_6mm_H5mm
- moved SW13 9.89 mm to (95.5, 17.0)
- moved J3 9.72 mm to (103.4, 32.5)
- moved TP5 9.72 mm to (101.3, 38.5)
- moved TP6 9.72 mm to (105.8, 38.5)
- moved R17 6.92 mm to (108.1, 20.6)
- moved J2 4.66 mm to (102.1, 70.6)
- moved J1 4.02 mm to (177.5, 47.8)
- moved SW10 4.02 mm to (173.0, 24.3)
- moved SW11 4.02 mm to (173.0, 15.1)
- moved SW9 4.02 mm to (173.0, 5.84)
- moved SW12 4.02 mm to (173.1, 33.5)
- moved RV10 2.71 mm to (165.3, 17.5)
- moved RV9 2.30 mm to (149.9, 17.5)

Commit message: new pcb
Parts:
- removed H4: MountingHole_GND, MountingHole:MountingHole_2.7mm_M2.5_Pad
- removed J3: Conn_01x02_Female, Connector_PinHeader_2.54mm:PinHeader_1x02_P2.54mm_Vertical
- removed RV10, RV11, RV9: R_POT, Potentiometer_THT:Potentiometer_Bourns_PTV09A-1_Single_Vertical
- removed TP5, TP6: TestPoint, TestPoint:TestPoint_THTPad_2.5x2.5mm_Drill1.2mm
- added +3V3: TestPoint, TestPoint:TestPoint_THTPad_2.5x2.5mm_Drill1.2mm, F.Cu at (101.0, 65.7)
- added +5V: TestPoint, TestPoint:TestPoint_THTPad_2.5x2.5mm_Drill1.2mm, F.Cu at (101.0, 75.2)
- added GND: TestPoint, TestPoint:TestPoint_THTPad_2.5x2.5mm_Drill1.2mm, F.Cu at (100.9, 70.5)
- added GND: MountingHole_GND, MountingHole:MountingHole_2.7mm_M2.5_Pad, F.Cu at (100.5, 53.5)
- added OLED Display: OLED, Display:OLED_SPI_128x32, F.Cu at (126.0, 63.0)
- added PWR: Conn_01x03_Female, Connector_PinHeader_2.54mm:PinHeader_1x03_P2.54mm_Vertical, F.Cu at (105.6, 65.8)
- added R18: R, Resistor_SMD:R_1806_4516Metric_Pad1.57x1.80mm_HandSolder, B.Cu at (188.1, 90.5)
- added R19: R, Resistor_SMD:R_1806_4516Metric_Pad1.57x1.80mm_HandSolder, B.Cu at (188.1, 62.8)
- added R20: R, Resistor_SMD:R_1806_4516Metric_Pad1.57x1.80mm_HandSolder, B.Cu at (173.3, 53.9)
- added R21: R, Resistor_SMD:R_1806_4516Metric_Pad1.57x1.80mm_HandSolder, B.Cu at (188.1, 72.0)
- added R22: R, Resistor_SMD:R_1806_4516Metric_Pad1.57x1.80mm_HandSolder, B.Cu at (188.1, 81.3)
- added SP1: R_POT, Potentiometer_THT:Potentiometer_Bourns_PTV09A-1_Single_Vertical, F.Cu at (154.1, 74.0)
- added SP2: R_POT, Potentiometer_THT:Potentiometer_Bourns_PTV09A-1_Single_Vertical, F.Cu at (169.8, 74.0)
- added SP3: R_POT, Potentiometer_THT:Potentiometer_Bourns_PTV09A-1_Single_Vertical, F.Cu at (109.2, 94.9)
- R9: moved to F.Cu
- moved R13 135.2 mm to (129.3, 135.3), turned to 90 degrees
- moved R17 125.6 mm to (159.6, 135.2), turned to 90 degrees
- moved R12 125.5 mm to (114.1, 135.5), turned to 270 degrees
- moved R16 119.4 mm to (144.6, 135.2), turned to 270 degrees
- moved R15 117.0 mm to (172.8, 112.2), turned to 270 degrees
- moved R14 106.5 mm to (157.0, 112.2), turned to 90 degrees
- moved R8 104.0 mm to (159.6, 103.8), turned to 90 degrees
- moved R11 103.7 mm to (132.2, 112.0), turned to 270 degrees
- moved R4 102.4 mm to (129.3, 103.9), turned to 90 degrees
- moved R3 98.8 mm to (114.1, 103.8), turned to 270 degrees
- moved R10 97.6 mm to (116.4, 112.1), turned to 90 degrees
- moved SSW5 96.0 mm to (183.1, 56.3), turned to 180 degrees
- moved R2 77.1 mm to (132.3, 80.7), turned to 270 degrees
- moved D9 74.3 mm to (161.2, 55.0), turned to 180 degrees
- moved R5 72.9 mm to (156.8, 80.9), turned to 90 degrees
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- renumbered SW12 to SSW1, SW10 to SSW2, SW11 to SSW3, SW9 to SSW4, SW13 to SSW5
Connections:
- J1 pad 1: R1 -> SP2
- J1 pad 10: L2 -> SSW1
- J1 pad 11: L3 -> SSW5
- J1 pad 12: L4 -> SSW3
- J1 pad 13: L5 -> +3V3
- J1 pad 14: L6 -> SSW2
- J1 pad 15: L7 -> L8
- J1 pad 16: L8 -> L7
- J1 pad 17: +5V -> R8
- J1 pad 18: GND -> R7
- J1 pad 19: NC -> B8
- J1 pad 2: R2 -> SP1
- J1 pad 20: NC -> B7
- J1 pad 3: R3 -> L4
- J1 pad 4: R4 -> L3
- J1 pad 5: R5 -> R4
- J1 pad 6: R6 -> R3
- J1 pad 7: R7 -> B4
- J1 pad 8: R8 -> B3
- J1 pad 9: L1 -> SSW4
- J2 pad 1: B1 -> SP3
- J2 pad 10: NC -> L1
- J2 pad 11: NC -> R2
- J2 pad 12: NC -> R1
- J2 pad 13: NC -> B2
- J2 pad 14: NC -> B1
- J2 pad 15: NC -> L6
- J2 pad 16: NC -> L5
- J2 pad 17: NC -> R6
- J2 pad 18: NC -> R5
- J2 pad 19: NC -> B6
- J2 pad 2: B2 -> GND
- J2 pad 20: NC -> B5
- J2 pad 3: B3 -> CLK
- J2 pad 4: B4 -> +5V
- J2 pad 5: B5 -> MOSI
- J2 pad 6: B6 -> RES
- J2 pad 7: B7 -> DC
- J2 pad 8: B8 -> CS
- J2 pad 9: NC -> L2
- SSW1 pad 1: NC -> +3V3
- SSW1 pad 2: NC -> SSW1
- SSW2 pad 1: NC -> +3V3
- SSW2 pad 2: NC -> SSW4
- SSW3 pad 1: NC -> +3V3
- SSW3 pad 2: NC -> SSW3
- SSW4 pad 1: NC -> +3V3
- SSW4 pad 2: NC -> SSW5
- SSW5 pad 1: NC -> SSW2
- SSW5 pad 2: NC -> +3V3
- SW1 pad 1: +5V -> +3V3
- SW2 pad 1: +5V -> +3V3
- SW3 pad 1: +5V -> +3V3
- SW4 pad 1: +5V -> +3V3
- SW5 pad 1: +5V -> +3V3
- SW6 pad 1: +5V -> +3V3
- SW7 pad 1: +5V -> +3V3
- SW8 pad 1: +5V -> +3V3
Routing:
- net +3V3: track 0.00 -> 305.4 mm
- net CS: track 0.00 -> 71.5 mm
- net SSW2: track 0.00 -> 71.0 mm
- net RES: track 0.00 -> 66.3 mm
- net DC: track 0.00 -> 65.4 mm
- net MOSI: track 0.00 -> 62.4 mm
- net CLK: track 0.00 -> 58.3 mm
- net SSW5: track 0.00 -> 57.3 mm
- net SSW3: track 0.00 -> 49.8 mm
- net L2: track 0.00 -> 49.4 mm
- net L1: track 0.00 -> 41.6 mm
- net SP1: track 0.00 -> 39.9 mm
- net R2: track 0.00 -> 37.9 mm
- net SSW4: track 0.00 -> 35.6 mm
- net B2: track 0.00 -> 35.4 mm
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- added copper zone on F.Cu, net +5V
- added copper zone on B.Cu, net GND
Other:
- board outline added: 95 x 90 mm
- board text added: "CV/MIDI Sequencer © Karl Johannes Jondell v. 0.01b / 290820"

Commit message: new led
Parts:
- D9: footprint LED_THT:LED_D5.0mm -> LED_SMD:LED_1206_3216Metric_Pad1.42x1.75mm_HandSolder
Routing:
- net GND: track 0.00 -> 20.6 mm
- net Net-(D9-Pad2): track 3.67 -> 4.72 mm

Commit message: new led
Parts:
- R1, R10, R11, R12, R13, R14, R15, R16, R17, R18, R19, R2, R20, R21, R22, R3, R4, R5, R6, R7, R8, R9: footprint Resistor_SMD:R_1806_4516Metric_Pad1.57x1.80mm_HandSolder -> Resistor_SMD:R_1206_3216Metric_Pad1.42x1.75mm_HandSolder
- RV1, RV2, RV3, RV4, RV5, RV6, RV7, RV8, SP1, SP2, SP3: footprint Potentiometer_THT:Potentiometer_Bourns_PTV09A-1_Single_Vertical -> Potentiometer_THT:Potentiometer_Alps_RK09K_Single_Vertical

Commit message: new pcb
Parts:
- removed R22: R, Resistor_SMD:R_1206_3216Metric_Pad1.42x1.75mm_HandSolder
- removed SP2: R_POT, Potentiometer_THT:Potentiometer_Alps_RK09K_Single_Vertical
- removed the SSW2 at (177.2, 79.0)
- removed SSW4: SW_Push, Button_Switch_THT:SW_PUSH_6mm_H5mm
- added SW9: Rotary_Encoder_Switch, Rotary_Encoder:RotaryEncoder_Alps_EC12E-Switch_Vertical_H20mm, F.Cu at (164.6, 74.4)
- OLED_Display1: renamed from OLED Display
- R1, R10, R11, R14, R15, R2, R5, R6, R9: value R -> 220
- R12, R13, R16, R17, R18, R19, R20, R21, R3, R4, R7, R8: value R -> 2k2
- SP1, SP3: value R_POT -> R_POT_SETTING
- moved R19 22.8 mm to (166.8, 54.8), turned to 0 degrees
- moved R20 17.5 mm to (188.2, 63.0)
- moved SSW2 8.93 mm to (183.8, 65.2)
- moved D9 5.80 mm to (155.4, 54.9)
- moved R9 5.80 mm to (147.2, 54.9)
- moved SSW3 4.67 mm to (177.3, 74.5)
- moved R21 4.57 mm to (188.0, 76.6)
- renumbered GND to H4, PWR to J3, SSW5 to SSW2, +3V3 to TP1, GND to TP2, +5V to TP3
Connections:
- J1 pad 1: SP2 -> RE2
- J1 pad 10: SSW1 -> RE1
- J1 pad 11: SSW5 -> SSW2
- J1 pad 14: SSW2 -> SSW4
- J1 pad 9: SSW4 -> SSW1
- R19 pad 1: SSW5 -> GND
- R19 pad 2: GND -> SSW4
Routing:
- net SSW5: track 57.5 -> 0.00 mm
- net RE1: track 0.00 -> 46.4 mm
- net SSW4: track 35.8 -> 82.0 mm
- net RE2: track 0.00 -> 35.2 mm
- net SP2: track 35.0 -> 0.00 mm
- net SSW2: track 71.2 -> 57.7 mm
- net +3V3: track 305.4 -> 300.4 mm
- net SSW3: track 50.0 -> 45.5 mm
- net SSW1: track 27.4 -> 25.3 mm
- net GND: track 20.6 -> 22.5 mm
- net Net-(D9-Pad2): track 4.72 -> 5.33 mm
Other:
- board text added: "CV/MIDI Sequencer © Karl Johannes Jondell v. 0.02b / 150920"
- board text removed: "CV/MIDI Sequencer © Karl Johannes Jondell v. 0.01b / 290820"

Commit message: cv expander
Parts:
- moved SSW2 1.55 mm to (183.8, 66.8)
- moved R20 1.50 mm to (188.2, 64.5)
- moved R21 0.90 mm to (188.0, 77.5)
- moved SSW3 0.77 mm to (177.3, 75.3)
Routing:
- net +3V3: track 300.4 -> 298.8 mm
- net SSW2: track 57.7 -> 56.3 mm
- net SSW4: track 82.0 -> 83.0 mm
Other:
- board text added: "CV/MIDI Sequencer © Karl Johannes Jondell v. 0.02b / 160920"
- board text added: "Power on (5V)"
- board text removed: "CV/MIDI Sequencer © Karl Johannes Jondell v. 0.02b / 150920"
